File: pathfinderKey-Cuts.kicad_pcb (KiCad board)
At the start: 2 copper layers, 78 x 60.5 mm, 13 parts, among them SW1 SW_Push, SW2 SW_Push, SW3 SW_Push, SW4 SW_Push, U1 XIAO-RP2040-DIP

Commit message: Add files via upload
Routing:
- net LED1: track 60.4 -> 202.7 mm
- net button1: track 47.9 -> 45.5 mm
Other:
- outline, holes or cut-outs redrawn
Changed lines of the file:
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@@
-		(layer "Edge.Cuts")
-	)
-	(gr_arc
-		(start 136 112)
-		(mid 136.177488 111.292213)
-		(end 136.66795 110.751925)
-		(stroke
-			(width 0.05)
-			(type default)
-		)
 		(layer "Edge.Cuts")
 	)
@@
 	)
 	(gr_line
+		(start 157.5 108)
+		(end 157.5 109.5)
+		(stroke
+			(width 0.05)
+			(type default)
+		)
+		(layer "Edge.Cuts")
+	)
+	(gr_line
+		(start 136 136.5)
+		(end 136 113)
+		(stroke
+			(width 0.05)
+			(type default)
+		)
+		(layer "Edge.Cuts")
+	)
+	(gr_line
 		(start 214 135.5)
 		(end 214 136.5)
@@
 	)
 	(gr_line
-		(start 156 102)
-		(end 146 102.085787)
+		(start 157.5 100.5)
+		(end 157.5 108)
+		(stroke
+			(width 0.05)
+			(type default)
+		)
+		(layer "Edge.Cuts")
+	)
+	(gr_line
+		(start 138 111)
+		(end 156 111)
+		(stroke
+			(width 0.05)
+			(type default)
+		)
+		(layer "Edge.Cuts")
+	)
+	(gr_arc
+		(start 136 113)
+		(mid 136.585786 111.585786)
+		(end 138 111)
 		(stroke
 			(width 0.05)
@@
 	)
 	(gr_line
-		(start 136.66795 110.751925)
-		(end 145 102.500001)
-		(stroke
-			(width 0.05)
-			(type default)
-		)
-		(layer "Edge.Cuts")
-	)
-	(gr_line
-		(start 136 136.5)
-		(end 136 112)
-		(stroke
-			(width 0.05)
-			(type default)
-		)
-		(layer "Edge.Cuts")
-	)
-	(gr_arc
-		(start 145 102.5)
-		(mid 145.458804 102.193437)
-		(end 146 102.085786)
-		(stroke
-			(width 0.05)
-			(type default)
-		)
-		(layer "Edge.Cuts")
-	)
-	(gr_line
 		(start 157.5 100.5)
 		(end 157.5 95)
@@
 		(layer "Edge.Cuts")
 	)
+	(gr_arc
+		(start 157.5 109.5)
+		(mid 157.06066 110.56066)
+		(end 156 111)
+		(stroke
+			(width 0.05)
+			(type default)
+		)
+		(layer "Edge.Cuts")
+	)
 	(gr_line
 		(start 159.5 78)
@@
 		(layer "Edge.Cuts")
 	)
-	(gr_arc
-		(start 157.5 100.5)
-		(mid 157.06066 101.56066)
-		(end 156 102)
-		(stroke
-			(width 0.05)
-			(type default)
-		)
-		(layer "Edge.Cuts")
-	)
 	(segment
 		(start 168.5 80.92)
@@
 	)
 	(segment
-		(start 159.5 104)
-		(end 146.5 104)
-		(width 0.2)
-		(layer "F.Cu")
-		(net 5)
-	)
-	(segment
-		(start 140.84737 123.92)
-		(end 138 121.07263)
-		(width 0.2)
-		(layer "F.Cu")
-		(net 5)
-	)
-	(segment
-		(start 141.925 123.92)
-		(end 140.84737 123.92)
-		(width 0.2)
-		(layer "F.Cu")
-		(net 5)
-	)
-	(segment
-		(start 146.5 104)
-		(end 138 112.5)
+		(start 139 123.5)
+		(end 139.42 123.92)
+		(width 0.2)
+		(layer "F.Cu")
+		(net 5)
+	)
+	(segment
+		(start 139.42 123.92)
+		(end 141.925 123.92)
+		(width 0.2)
+		(layer "F.Cu")
+		(net 5)
+	)
+	(segment
+		(start 168.601 79)
+		(end 212.5 79)
+		(width 0.2)
+		(layer "F.Cu")
+		(net 5)
+	)
+	(segment
+		(start 167.499 84.999)
+		(end 167.499 80.102)
 		(width 0.2)
 		(layer "F.Cu")
@@
 	(segment
 		(start 168.5 86)
-		(end 159.5 95)
-		(width 0.2)
-		(layer "F.Cu")
-		(net 5)
-	)
-	(segment
-		(start 138 121.07263)
-		(end 138 112.5)
-		(width 0.2)
-		(layer "F.Cu")
-		(net 5)
-	)
-	(segment
-		(start 159.5 95)
-		(end 159.5 104)
+		(end 167.499 84.999)
+		(width 0.2)
+		(layer "F.Cu")
+		(net 5)
+	)
+	(segment
+		(start 212.5 136.5)
+		(end 211.5 137.5)
+		(width 0.2)
+		(layer "F.Cu")
+		(net 5)
+	)
+	(segment
+		(start 137.5 136.5)
+		(end 137.5 123.5)
+		(width 0.2)
+		(layer "F.Cu")
+		(net 5)
+	)
+	(segment
+		(start 212.5 79)
+		(end 212.5 136.5)
+		(width 0.2)
+		(layer "F.Cu")
+		(net 5)
+	)
+	(segment
+		(start 137.5 123.5)
+		(end 139 123.5)
+		(width 0.2)
+		(layer "F.Cu")
+		(net 5)
+	)
+	(segment
+		(start 211.5 137.5)
+		(end 138.5 137.5)
+		(width 0.2)
+		(layer "F.Cu")
+		(net 5)
+	)
+	(segment
+		(start 138.5 137.5)
+		(end 137.5 136.5)
+		(width 0.2)
+		(layer "F.Cu")
+		(net 5)
+	)
+	(segment
+		(start 167.499 80.102)
+		(end 168.601 79)
 		(width 0.2)
 		(layer "F.Cu")
@@
 	)
 	(segment
-		(start 167.91747 95.799)
-		(end 163.701 95.799)
+		(start 165 106.5)
+		(end 160 111.5)
 		(width 0.2)
 		(layer "F.Cu")
@@
 	)
 	(segment
-		(start 147.5 106)
-		(end 141.925 111.575)
+		(start 174.19847 91.92)
+		(end 165 101.11847)
 		(width 0.2)
 		(layer "F.Cu")
@@
 	)
 	(segment
-		(start 168.044578 95.926108)
-		(end 167.91747 95.799)
+		(start 175.04 91.92)
+		(end 174.19847 91.92)
 		(width 0.2)
 		(layer "F.Cu")
@@
 	)
 	(segment
-		(start 161 98.5)
-		(end 161 106)
+		(start 153.26 113.76)
+		(end 141.925 113.76)
 		(width 0.2)
 		(layer "F.Cu")
@@
 	)
 	(segment
-		(start 169.205206 95.926108)
-		(end 168.044578 95.926108)
+		(start 165 101.11847)
+		(end 165 106.5)
 		(width 0.2)
 		(layer "F.Cu")
@@
 	)
 	(segment
-		(start 175.04 91.92)
-		(end 173.211314 91.92)
+		(start 160 111.5)
+		(end 156 111.5)
 		(width 0.2)
 		(layer "F.Cu")
@@
 	)
 	(segment
-		(start 173.211314 91.92)
-		(end 169.205206 95.926108)
+		(start 153.5 114)
+		(end 153.26 113.76)
 		(width 0.2)
 		(layer "F.Cu")
@@
 	)
 	(segment
-		(start 161 106)
-		(end 147.5 106)
-		(width 0.2)
-		(layer "F.Cu")
-		(net 8)
-	)
-	(segment
-		(start 163.701 95.799)
-		(end 161 98.5)
-		(width 0.2)
-		(layer "F.Cu")
-		(net 8)
-	)
-	(segment
-		(start 141.925 111.575)
-		(end 141.925 113.76)
-		(width 0.2)
-		(layer "F.Cu")
+		(start 156 111.5)
+		(end 153.5 114)
+		(width 0.2)
+		(layer "F.Cu")

Commit message: Add files via upload
Parts:
- moved R4 41.5 mm to (154.0, 114.5)
- moved R2 40.7 mm to (154.5, 84.4)
- moved D4 39.5 mm to (160.5, 117.0)
- moved D2 39.4 mm to (160.5, 87.0)
- moved SW4 38.9 mm to (163.4, 126.4)
- moved SW2 38.4 mm to (163.4, 96.4)
- moved U1 17.3 mm to (134.9, 130.5)
- moved SW3 14.6 mm to (187.5, 126.4)
- moved SW1 13.3 mm to (187.5, 96.4)
- moved D3 13.3 mm to (184.8, 117.0)
- moved D1 12.1 mm to (184.8, 87.0)
- moved R3 12.1 mm to (178.6, 114.4)
- moved R1 10.5 mm to (178.6, 83.9)
Routing:
- net button4: track 206.5 -> 55.6 mm
- net button2: track 149.7 -> 57.3 mm
- net LED4: track 102.1 -> 28.8 mm
- net button1: track 45.5 -> 115.8 mm
- net LED1: track 202.7 -> 147.5 mm
- net button3: track 36.4 -> 74.2 mm
- net GND: track 161.7 -> 142.3 mm
- net LED3: track 88.7 -> 74.7 mm
- net LED2: track 163.3 -> 152.7 mm
- net Net-(D1-PadA): track 7.07 -> 8.78 mm
- net Net-(D3-PadA): track 7.15 -> 8.57 mm
- net Net-(D2-PadA): track 7.07 -> 8.34 mm
Other:
- board size 78 x 60.5 mm -> 81 x 71 mm
- board text added: "?"
